File: Feather-5 - Spring/LooUQ CircuitRiver - Feather-5 Spring.brd (EAGLE design)
At the start: 102.5 x 70.7 mm, 11 parts, among them J1 FEATHERHOST-S, J2 FEATHERHOST-L, J3 CR-SPRING HEADER, J4 JST PH-2 T/H, J5 JST PH-2 T/H, J6 QWIIC VERTICAL, J7 CR-RAPIDSIO VERTICAL, J8 DNF, P3 SLEEP

Commit message: Updated Feathers
Parts:
- added P1, P2: DNF, common:BreakoutConn
- P3: value SLEEP -> DNF
- moved J8 2.52 mm to (73.0, 59.7)
Connections:
- new net Net_0: J2.16, P1.1
- new net Net_24: J2.14, J8.1
- net Net_3v3: now also J8.2; no longer J8.1
- net Net_GND: now also P2.1; no longer J8.2
Routing:
- net Net_0: track 0.00 -> 27.3 mm
- net Net_24: track 0.00 -> 26.2 mm
- net Net_3v3: track 49.4 -> 43.3 mm
Other:
- board text added: "A.Ref"
- board text added: "MCU"
- board text removed: "GND"
Changed lines of the file:
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@@
 <rectangle x1="63.183" y1="32.385" x2="66.516" y2="27.94" layer="29" rot="R0"/>
 <rectangle x1="41.751" y1="43.18" x2="45.72" y2="40.005" layer="29" rot="R0"/>
-<text x="76.966" y="59.312" size="0.74" layer="21" font="proportional" ratio="10" rot="R0" align="top-left" distance="50">3v3</text>
-<text x="76.966" y="61.217" size="0.74" layer="21" font="proportional" ratio="10" rot="R0" align="top-left" distance="50">GND</text>
+<text x="74.208" y="61.344" size="0.74" layer="21" font="proportional" ratio="10" rot="R0" align="top-left" distance="50">3v3</text>
+<text x="74.305" y="59.378" size="0.74" layer="21" font="proportional" ratio="10" rot="R0" align="top-left" distance="50">A.Ref</text>
 <text x="56.964" y="62.487" size="0.74" layer="21" font="proportional" ratio="10" rot="R0" align="top-left" distance="50">Antenna Power</text>
 <text x="58.027" y="63.598" size="0.74" layer="21" font="proportional" ratio="10" rot="R0" align="top-left" distance="50">GPS Active</text>
 <text x="15.203" y="70.142" size="1.48" layer="21" font="proportional" ratio="10" rot="R0" align="top-left" distance="50">Important Connect Power to J5</text>
 <text x="15.203" y="67.66" size="1.48" layer="21" font="proportional" ratio="10" rot="R0" align="top-left" distance="50">or USB to Feather, not both.</text>
+<text x="71.443" y="69.035" size="0.74" layer="21" font="proportional" ratio="10" rot="R0" align="top-left" distance="50">MCU</text>
 </plain>
 <attributes/>
@@
 <attribute name="DESCRIPTION" value="CONN HEADER SMD 10POS 1MM" x="81.208733" y="65.246267" size="1.778" layer="27" display="off"/>
 </element>
-<element name="J8" library="common" package="HDR-1x2T/2/4x2" value="DNF" x="75.565" y="59.7375" rot="R90">
-<attribute name="NAME" value="J8" layer="21" x="73.046372" y="58.98437" size="0.814" align="top-left" rot="R0"/>
-<attribute name="MANUFACTURER" value="3M" x="75.565" y="59.7375" size="1.778" layer="27" display="off"/>
-<attribute name="DATASHEET" value="https://media.digikey.com/pdf/Data%20Sheets/3M%20PDFs/951yyy-xx22-AR_Series%20Datasheet.pdf" x="75.565" y="59.7375" size="1.778" layer="27" display="off"/>
-<attribute name="MFGPARTNM" value="951102-8622-AR" x="75.565" y="59.7375" size="1.778" layer="27" display="off"/>
-</element>
-<element name="LG1" library="common" package="LooUQ-6mm" value="LOOUQ LOGO" x="85.4075" y="3.913156" rot="R0"/>
+<element name="J8" library="common" package="HDR-1x2T/2/4x2" value="DNF" x="73.048665" y="59.7375" rot="R90">
+<attribute name="NAME" value="J8" layer="21" x="70.530037" y="58.98437" size="0.814" align="top-left" rot="R0"/>
+<attribute name="MANUFACTURER" value="3M" x="73.048665" y="59.7375" size="1.778" layer="27" display="off"/>
+<attribute name="DATASHEET" value="https://media.digikey.com/pdf/Data%20Sheets/3M%20PDFs/951yyy-xx22-AR_Series%20Datasheet.pdf" x="73.048665" y="59.7375" size="1.778" layer="27" display="off"/>
+<attribute name="MFGPARTNM" value="951102-8622-AR" x="73.048665" y="59.7375" size="1.778" layer="27" display="off"/>
+</element>
+<element name="LG1" library="common" package="LooUQ-6mm" value="LOOUQ LOGO" x="85.4075" y="3.913121" rot="R0"/>
 <element name="LG2" library="common" package="CircuitRiver-6mm" value="CIRCUITRIVER LOGO" x="87.788767" y="50.641233" rot="MR-90"/>
-<element name="P3" library="common" package="BreakoutConn" value="SLEEP" x="45.561233" y="5.3975" rot="R90">
+<element name="P1" library="common" package="BreakoutConn" value="DNF" x="73.423387" y="65.527801" rot="R90">
+<attribute name="NAME" value="~RESET" layer="21" x="70.735511" y="67.85378" size="0.814" align="top-left" rot="R0"/>
+</element>
+<element name="P2" library="common" package="BreakoutConn" value="DNF" x="79.065753" y="60.495131" rot="R90">
+<attribute name="NAME" value="GND" layer="21" x="77.939477" y="62.579155" size="0.814" align="top-left" rot="R0"/>
+</element>
+<element name="P3" library="common" package="BreakoutConn" value="DNF" x="45.561233" y="5.3975" rot="R90">
 <attribute name="NAME" value="Sleep" layer="21" x="44.120445" y="7.77187" size="0.814" align="top-left" rot="R0"/>
 </element>
@@
 <signal name="S$2" class="0">
 <via x="40.9575" y="6.35" extent="1-16" drill="0.4" diameter="0.8" shape="round" alwaysstop="no"/>
+</signal>
+<signal name="Net_0">
+<contactref element="J2" pad="16"/>
+<contactref element="P1" pad="1"/>
+<wire layer="1" width="0.2" x1="73.423387" y1="65.527801" x2="71.627763" y2="65.527801"/>
+<wire layer="1" width="0.2" x1="71.627763" y1="65.527801" x2="69.103127" y2="63.003165"/>
+<wire layer="1" width="0.2" x1="69.103127" y1="63.003165" x2="48.715665" y2="63.003165"/>
+<wire layer="1" width="0.2" x1="48.715665" y1="63.003165" x2="47.625" y2="61.9125"/>
 </signal>
 <signal name="Net_1">
@@
 <wire layer="1" width="0.2" x1="81.661667" y1="65.246267" x2="81.708733" y2="65.246267"/>
 </signal>
+<signal name="Net_24">
+<contactref element="J2" pad="14"/>
+<contactref element="J8" pad="1"/>
+<wire layer="1" width="0.2" x1="73.048665" y1="58.7375" x2="49.53" y2="58.7375"/>
+<wire layer="1" width="0.2" x1="49.53" y1="58.7375" x2="47.625" y2="56.8325"/>
+</signal>
 <signal name="Net_25">
 <contactref element="J2" pad="11"/>
@@
 <contactref element="J6" pad="2"/>
 <contactref element="J7" pad="2"/>
-<contactref element="J8" pad="1"/>
-<wire layer="1" width="0.5" x1="83.708733" y1="58.578767" x2="83.708733" y2="59.777"/>
-<wire layer="1" width="0.5" x1="83.708733" y1="59.777" x2="76.6045" y2="59.777"/>
-<wire layer="1" width="0.5" x1="76.6045" y1="59.777" x2="75.565" y2="58.7375"/>
-<wire layer="1" width="1" x1="47.625" y1="59.3725" x2="57.524433" y2="59.3725"/>
-<wire layer="1" width="1" x1="57.524433" y1="59.3725" x2="58.662733" y2="58.7375"/>
-<wire layer="1" width="1" x1="58.662733" y1="58.7375" x2="75.565" y2="58.7375"/>
+<contactref element="J8" pad="2"/>
 <wire layer="1" width="0.5" x1="77.708733" y1="65.246267" x2="77.708733" y2="63.448433"/>
-<wire layer="1" width="0.5" x1="77.708733" y1="63.448433" x2="78.417867" y2="62.7393"/>
+<wire layer="1" width="0.5" x1="77.708733" y1="63.448433" x2="77.797538" y2="63.359629"/>
+<wire layer="1" width="0.5" x1="77.797538" y1="63.359629" x2="78.417867" y2="62.7393"/>
 <wire layer="1" width="0.5" x1="78.417867" y1="62.7393" x2="82.2642" y2="62.7393"/>
 <wire layer="1" width="0.5" x1="82.2642" y1="62.7393" x2="83.708733" y2="61.562467"/>
 <wire layer="1" width="0.5" x1="83.708733" y1="61.562467" x2="83.708733" y2="58.578767"/>
+<wire layer="1" width="0.5" x1="73.048665" y1="60.7375" x2="48.99" y2="60.7375"/>
+<wire layer="1" width="0.5" x1="48.99" y1="60.7375" x2="47.625" y2="59.3725"/>
+<wire layer="1" width="0.5" x1="73.048665" y1="60.7375" x2="75.175409" y2="60.7375"/>
+<wire layer="1" width="0.5" x1="75.175409" y1="60.7375" x2="77.797538" y2="63.359629"/>
 </signal>
 <signal name="Net_GND" class="1">
@@
 <contactref element="J6" pad="1"/>
 <contactref element="J7" pad="1"/>
-<contactref element="J8" pad="2"/>
+<contactref element="P2" pad="1"/>
 <via x="78.105" y="54.9275" extent="1-16" drill="0.4" diameter="0.8" shape="round" alwaysstop="no"/>
-<via x="73.818733" y="60.6425" extent="1-16" drill="0.4" diameter="0.8" shape="round" alwaysstop="no"/>
-<via x="77.311267" y="60.6425" extent="1-16" drill="0.4" diameter="0.8" shape="round" alwaysstop="no"/>
 <polygon width="0.635" layer="16" spacing="1.27" isolate="0.33" thermals="no">
 <vertex x="9.8425" y="69.85"/>

Commit message: Moved RapidsIO, chg L1 on F-630
Parts:
- J4: value JST PH-2 T/H -> JST PH-2 R/A T/H; device common:JST_PH-2_T/H -> common:JST_PH-2_R/A_T/H
- J5: value JST PH-2 T/H -> JST PH-2 VERT T/H; device common:HDR-2x1T/2x2/2x4 -> common:JST_PH-2_VERT_T/H
- J6: device common:JST-SH_SMD-TopEntry_Qwiic -> common:JST_SH-04_VERT_SMD_Qwiic
- J7: device common:JST-SH_SMD-TopEntry_Rapids -> common:JST_SH-10_VERT_SMD_RapidsIO
- LG1: value LOOUQ LOGO -> DNF
- LG2: value CIRCUITRIVER LOGO -> DNF
- moved J5 85.3 mm to (97.4, 55.3)
- moved LG1 77.6 mm to (38.8, 66.0)
- moved J4 49.7 mm to (13.0, 66.1), turned to 0 degrees
- moved J6 36.9 mm to (73.4, 23.3), turned to 90 degrees
- moved J7 31.6 mm to (73.3, 34.7), turned to 90 degrees
- moved P1 26.7 mm to (88.6, 43.5)
- moved P2 18.2 mm to (85.2, 43.4)
- moved J8 18.1 mm to (80.9, 43.4), turned to 0 degrees
- moved LG2 10.2 mm to (97.5, 47.5)
Routing:
- net Net_VBAT: track 127.4 -> 175.4 mm
- net Net_27: track 46.4 -> 5.53 mm
- net Net_28: track 40.7 -> 6.06 mm
- net Net_8: track 123.7 -> 89.9 mm, vias 1 -> 2
- net Net_6: track 130.7 -> 97.5 mm, vias 3 -> 4
- net Net_2: track 133.4 -> 100.9 mm, vias 3 -> 4
- net Net_3v3: track 43.3 -> 74.5 mm
- net Net_VBUS: track 73.5 -> 44.0 mm, vias 2 -> 0
- net Net_0: track 27.3 -> 49.3 mm
- net Net_11: track 39.3 -> 60.3 mm, vias 1 -> 0
- net Net_25: track 41.3 -> 59.4 mm, vias 1 -> 0
- net Net_15: track 44.2 -> 59.2 mm, vias 1 -> 0
- net Net_23: track 47.2 -> 60.1 mm, vias 1 -> 0
- net Net_24: track 26.2 -> 38.1 mm
- net Net_18: track 50.0 -> 60.2 mm, vias 1 -> 0
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- removed copper zone on layer 1, net Net_18
Other:
- board text added: "6v-30v DC"
- board text added: "Connect Power to PowerIn (J5)"
- board text added: "F.Batt"
- board text added: "Feather-5 Spring v1.5a"
- board text added: "GPS/GNSS Active"
- board text added: "Important"
- board text added: "PowerIn"
- board text removed: "F.Pwr"
- board text removed: "Feather-5 Spring v1.5"
- board text removed: "GPS Active"
- board text removed: "Important Connect Power to J5"
